File: TP_Buck_LT1959/TP_Buck_LT1959.kicad_pcb (KiCad board)
At the start: 2 copper layers, 185 x 126 mm, 56 parts, among them IC1 LT1959CS8#PBF, J1 Conn_01x02, T1 PA1005.100NL, T2 PA1005.100NL

Commit message: update PCB Buck et TD
Parts:
- D5: value MBR0540-TP -> STPS1L40ZFY
- F1: value SMD1812B075TF -> SMD1812B075TF/33

Commit message: Update TD
Parts:
- D5: value STPS1L40ZFY -> PMEG40T20ERX
- R5: value 47 -> 5.7
- R7: value 5.6 -> 47
- TP1: value i_c- -> i_c+
- TP2: value i_c+ -> i_c-
- TP8: value i_l- -> i_l+
- TP9: value i_l+ -> i_l-
