File: TP_Buck_LT1959/TP_Buck_LT1959.kicad_sch (KiCad schematic)
At the start: 53 parts, among them IC1 LT1959CS8#PBF, J1 Conn_01x02, T1 PA1005.100NL, T2 PA1005.100NL

Commit message: update PCB Buck et TD
Parts:
- D5: value MBR0540-TP -> PMEG40T20ERX
- F1: value SMD1812B075TF -> SMD1812B075TF/33
Changed lines of the file:
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@@
 	(title_block
 		(title "TP Buck (LT1959)")
-		(date "2026-06-01")
+		(date "2026-06-19")
 		(rev "V2")
 		(company "ENSEA")
@@
 			)
 		)
-		(property "Value" "MBR0540-TP"
+		(property "Value" "PMEG40T20ERX"
 			(at 204.7875 127 0)
 			(effects
@@
 			)
 		)
-		(property "Value" "SMD1812B075TF"
+		(property "Value" "SMD1812B075TF/33"
 			(at 229.87 127 90)
 			(effects

Commit message: Update TD
Parts:
- R5: value 47 -> 5.7
- R7: value 5.6 -> 47
- TP1: value i_c- -> i_c+
- TP2: value i_c+ -> i_c-
- TP8: value i_l- -> i_l+
- TP9: value i_l+ -> i_l-
Changed lines of the file:
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@@
 	(title_block
 		(title "TP Buck (LT1959)")
-		(date "2026-06-19")
+		(date "2026-06-22")
 		(rev "V2")
 		(company "ENSEA")
@@
 			)
 		)
-		(property "Value" "i_l-"
+		(property "Value" "i_l+"
 			(at 187.452 76.708 0)
 			(effects
@@
 			)
 		)
-		(property "Value" "i_l+"
+		(property "Value" "i_l-"
 			(at 198.628 76.708 0)
 			(effects
@@
 			)
 		)
-		(property "Value" "47"
+		(property "Value" "5.7"
 			(at 144.78 148.5899 90)
 			(effects
@@
 			)
 		)
-		(property "Value" "i_c-"
+		(property "Value" "i_c+"
 			(at 32.512 111.252 0)
 			(effects
@@
 			)
 		)
-		(property "Value" "i_c+"
+		(property "Value" "i_c-"
 			(at 32.512 122.428 0)
 			(effects
@@
 			)
 		)
-		(property "Value" "5.6"
+		(property "Value" "47"
 			(at 128.27 148.5899 90)
 			(effects
