File: Maquette_TP_Buck_LT1959/TP_Buck_LT1959.kicad_pcb (KiCad board)
At the start: 2 copper layers, 185 x 126 mm, 56 parts, among them IC1 LT1959CS8#PBF, J1 Conn_01x02, T1 PA1005.100NL, T2 PA1005.100NL

Commit message: Update 2026 (CM + TD)
Parts:
- L3: value 680u -> 270u
