File: Maquette_TP_Buck_LT1959/TP_Buck_LT1959.kicad_sch (KiCad schematic)
At the start: 53 parts, among them IC1 LT1959CS8#PBF, J1 Conn_01x02, T1 PA1005.100NL, T2 PA1005.100NL

Commit message: Update 2026 (CM + TD)
Parts:
- L3: value 680u -> 270u
Changed lines of the file:
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@@
 			)
 		)
-		(property "Value" "680u"
+		(property "Value" "270u"
 			(at 172.72 47.498 90)
 			(effects
